Commit message: three extra envs

File: urdf/ant_torso.urdf (robot description, URDF)
Before this commit: robot , 22 links, 21 joints
Links:
- removed link base_link
- link aux_1: geometry collision cylinder length=0.28284 radius=0.08000
- link aux_2: geometry collision cylinder length=0.28284 radius=0.08000
- link aux_3: geometry collision cylinder length=0.28284 radius=0.08000
- link aux_4: geometry collision cylinder length=0.28284 radius=0.08000
- link front_left_foot: geometry collision cylinder length=0.56569 radius=0.08000
- link front_left_leg: geometry collision cylinder length=0.28284 radius=0.08000
- link front_right_foot: geometry collision cylinder length=0.56569 radius=0.08000
- link front_right_leg: geometry collision cylinder length=0.28284 radius=0.08000
- link left_back_foot: geometry collision cylinder length=0.56569 radius=0.08000
- link left_back_leg: geometry collision cylinder length=0.28284 radius=0.08000
- link right_back_foot: geometry collision cylinder length=0.56569 radius=0.08000
- link right_back_leg: geometry collision cylinder length=0.28284 radius=0.08000
- link torso: geometry collision sphere radius=0.25000
Joints:
- removed joint base_to_torso
- joint ankle_1: limit lower=-0.50000 upper=0.50000 effort=1000.0 velocity=0.5 -> (none)
- joint ankle_2: limit lower=-0.50000 upper=0.50000 effort=1000.0 velocity=0.5 -> (none)
- joint ankle_3: limit lower=-0.50000 upper=0.50000 effort=1000.0 velocity=0.5 -> (none)
- joint ankle_4: limit lower=-0.50000 upper=0.50000 effort=1000.0 velocity=0.5 -> (none)
- joint hip_1: limit lower=-0.50000 upper=0.50000 effort=1000.0 velocity=0.5 -> (none)
- joint hip_2: limit lower=-0.50000 upper=0.50000 effort=1000.0 velocity=0.5 -> (none)
- joint hip_3: limit lower=-0.50000 upper=0.50000 effort=1000.0 velocity=0.5 -> (none)
- joint hip_4: limit lower=-0.50000 upper=0.50000 effort=1000.0 velocity=0.5 -> (none)

File: urdf/hopper.urdf (robot description, URDF)
Before this commit: robot , 5 links, 4 joints
Links:
- removed link base_link
Joints:
- removed joint base_to_slide
- removed joint leg_to_foot_joint
- removed joint thigh_to_leg_joint
- removed joint torso_to_thigh_joint
- added joint foot_joint: type revolute, parent leg, child foot, origin xyz=0.00000 0.00000 0.00000 rpy=0.00000 -0.00000 0.00000, axis 0.00000 1.00000 0.00000, limit lower=-0.50000 upper=0.50000 effort=1000.0 velocity=0.5
- added joint leg_joint: type revolute, parent thigh, child leg, origin xyz=0.00000 0.00000 0.00000 rpy=0.00000 -0.00000 0.00000, axis 0.00000 1.00000 0.00000, limit lower=-0.50000 upper=0.50000 effort=1000.0 velocity=0.5
- added joint thigh_joint: type revolute, parent torso, child thigh, origin xyz=0.00000 0.00000 0.00000 rpy=0.00000 -0.00000 0.00000, axis 0.00000 1.00000 0.00000, limit lower=-0.50000 upper=0.50000 effort=1000.0 velocity=0.5

File: urdf/hopper_link_0_1.urdf (robot description, URDF)
Before this commit: robot , 7 links, 6 joints
Links:
- removed link link0_1
- removed link link0_2
- removed link link0_3
- removed link link0_4
- removed link link0_6
- added link foot, mass 5.31557; collision cylinder length=0.39000 radius=0.06000; visual cylinder length=0.39000 radius=0.06000
- added link leg, mass 2.78136; collision cylinder length=0.50000 radius=0.04000; visual cylinder length=0.50000 radius=0.04000
Joints:
- removed joint ignore1
- removed joint ignore2
- removed joint ignore3
- removed joint jointfix_2_6
- removed joint jointfix_3_4
- added joint foot_joint: type revolute, parent leg, child foot, origin xyz=0.00000 0.00000 0.00000 rpy=0.00000 -0.00000 0.00000, axis 0.00000 1.00000 0.00000, limit lower=-0.50000 upper=0.50000 effort=1000.0 velocity=0.5
- added joint leg_joint: type revolute, parent thigh, child leg, origin xyz=0.00000 0.00000 0.00000 rpy=0.00000 -0.00000 0.00000, axis 0.00000 1.00000 0.00000, limit lower=-0.50000 upper=0.50000 effort=1000.0 velocity=0.5
- joint thigh_joint: child link0_6 -> thigh; origin xyz=0.00000 0.00000 1.05000 rpy=0.00000 -0.00000 0.00000 -> xyz=0.00000 0.00000 0.00000 rpy=0.00000 -0.00000 0.00000
