Commit message: inverted_pendulum urdf

File: urdf/hopper.urdf (robot description, URDF)
Before this commit: robot , 12 links, 11 joints
Links:
- removed link foot
- removed link leg
- removed link link0_10
- removed link link0_8
- removed link thigh
- link link0_6: geometry visual box size=0.08 0.08 1.0
Joints:
- removed joint foot_joint
- removed joint jointfix_0_10
- removed joint jointfix_1_8
- removed joint jointfix_2_6
- removed joint leg_joint

Commit message: render hopper

File: urdf/hopper.urdf (robot description, URDF)
Before this commit: robot , 7 links, 6 joints
Links:
- removed link link0_1
- removed link link0_2
- removed link link0_3
- removed link link0_4
- removed link link0_6
- added link foot, mass 5.31557; collision cylinder length=0.39000 radius=0.06000; visual cylinder length=0.39000 radius=0.06000
- added link leg, mass 2.78136; collision cylinder length=0.50000 radius=0.04000; visual cylinder length=0.50000 radius=0.04000
- added link thigh, mass 4.05789; collision cylinder length=0.45000 radius=0.05000; visual cylinder length=0.45000 radius=0.05000
Joints:
- removed joint ignore1
- removed joint ignore2
- removed joint ignore3
- removed joint jointfix_3_4
- removed joint thigh_joint
- added joint leg_to_foot_joint: type revolute, parent leg, child foot, origin xyz=0.00000 0.00000 -0.10000 rpy=0.00000 -0.00000 0.00000, axis 0.00000 1.00000 0.00000, limit lower=-0.50000 upper=0.50000 effort=1000.0 velocity=0.5
- added joint thigh_to_leg_joint: type revolute, parent thigh, child leg, origin xyz=0.00000 0.00000 -0.60000 rpy=0.00000 -0.00000 0.00000, axis 0.00000 1.00000 0.00000, limit lower=-0.50000 upper=0.50000 effort=1000.0 velocity=0.5
- added joint torso_to_thigh_joint: type revolute, parent torso, child thigh, origin xyz=0.00000 0.00000 -1.05000 rpy=0.00000 -0.00000 0.00000, axis 0.00000 1.00000 0.00000, limit lower=-0.50000 upper=0.50000 effort=1000.0 velocity=0.5
- joint base_to_slide: child link0_1 -> torso

Commit message: hopper main

File: urdf/hopper.urdf (robot description, URDF)
Before this commit: robot , 4 links, 3 joints
Links:
- added link base_link, mass 0.1
Joints:
- added joint base_to_torso: type continuous, parent base_link, child torso, origin xyz=0 0 1.0 rpy=0 0 0
