Commit message: add gym-like cartpole env

File: urdf/inverted pendulum_link1_1.urdf (robot description, URDF)
Before this commit: robot , 4 links, 3 joints
Links:
- link cart: mass 10.47198 -> 0.4
- link pole: mass 5.01859 -> 0.3; geometry collision cylinder length=0.60000 radius=0.04900; visual cylinder length=4.0 radius=0.04900
